Commit message: Imported upstream version '1.0.1' of 'upstream'

File: end_effectors/common/franka_hand.xacro (robot description, xacro)
@@ -2,5 +2,17 @@
 <robot xmlns:xacro="http://www.ros.org/wiki/xacro" name="hand">
   <!-- safety_distance: Minimum safety distance in [m] by which the collision volumes are expanded and which is enforced during robot motions -->
-  <xacro:macro name="franka_hand" params="connected_to:='' arm_id arm_prefix:='' ee_id ee_inertials rpy_ee:='0 0 0' xyz_ee:='0 0 0' tcp_xyz:='0 0 0.1034' tcp_rpy:='0 0 0' safety_distance:=0 gazebo:=false description_pkg:=franka_description with_sc:=false">
+  <xacro:macro name="franka_hand"
+               params="connected_to:=''
+                       arm_id arm_prefix:=''
+                       ee_id ee_inertials
+                       rpy_ee:='0 0 0'
+                       xyz_ee:='0 0 0'
+                       tcp_xyz:='0 0 0.1034'
+                       tcp_rpy:='0 0 0'
+                       safety_distance:=0
+                       gazebo:=false
+                       description_pkg:=franka_description
+                       with_sc:=false
+                       no_prefix:=false">
     <xacro:property name="ee_prefix" default="robot_"/>
     <xacro:unless value="${arm_id == ''}">
@@ -61,11 +73,9 @@
         </geometry>
       </collision>
-      <xacro:if value="${gazebo}">
-        <xacro:ee-inertials name="leftfinger" />
-      </xacro:if>
+      <xacro:ee-inertials name="leftfinger" />
     </link>
     <link name="${ee_prefix}rightfinger">
       <visual name="${ee_prefix}rightfinger_visual">
-        <origin xyz="0 0 0" rpy="0 0 ${pi}" />
+        <origin xyz="0 0 0" rpy="0 0 0" />
         <geometry>
           <mesh filename="package://${description_pkg}/meshes/robot_ee/${ee_id}/visual/finger.dae" />
@@ -74,5 +84,5 @@
       <!-- screw mount -->
       <collision>
-        <origin xyz="0 -18.5e-3 11e-3" rpy="0 0 0" />
+        <origin xyz="0 18.5e-3 11e-3" rpy="0 0 0" />
         <geometry>
           <box size="22e-3 15e-3 20e-3" />
@@ -81,5 +91,5 @@
       <!-- cartriage sledge -->
       <collision>
-        <origin xyz="0 -6.8e-3 2.2e-3" rpy="0 0 0" />
+        <origin xyz="0 6.8e-3 2.2e-3" rpy="0 0 0" />
         <geometry>
           <box size="22e-3 8.8e-3 3.8e-3" />
@@ -88,5 +98,5 @@
       <!-- diagonal finger -->
       <collision>
-        <origin xyz="0 -15.9e-3 28.35e-3" rpy="${-pi/6} 0 0" />
+        <origin xyz="0 15.9e-3 28.35e-3" rpy="${-pi/6} 0 ${pi}" />
         <geometry>
           <box size="17.5e-3 7e-3 23.5e-3" />
@@ -95,12 +105,10 @@
       <!-- rubber tip with which to grasp -->
       <collision>
-        <origin xyz="0 -7.58e-3 45.25e-3" rpy="0 0 0" />
+        <origin xyz="0 7.58e-3 45.25e-3" rpy="0 0 0" />
         <geometry>
           <box size="17.5e-3 15.2e-3 18.5e-3" />
         </geometry>
       </collision>
-      <xacro:if value="${gazebo}">
-        <xacro:ee-inertials name="rightfinger" />
-      </xacro:if>
+      <xacro:ee-inertials name="rightfinger" />
     </link>
     <joint name="${ee_prefix}finger_joint1" type="prismatic">
@@ -115,6 +123,6 @@
       <parent link="${ee_prefix}hand" />
       <child link="${ee_prefix}rightfinger" />
-      <origin xyz="0 0 0.0584" rpy="0 0 0" />
-      <axis xyz="0 -1 0" />
+      <origin xyz="0 0 0.0584" rpy="0 0 ${pi}" />
+      <axis xyz="0 1 0" />
       <limit effort="100" lower="0.0" upper="0.04" velocity="0.2" />
       <mimic joint="${ee_prefix}finger_joint1" />

File: robots/common/franka_arm.ros2_control.xacro (robot description, xacro)
@@ -3,15 +3,15 @@
 <xacro:macro name="franka_arm_ros2_control"
          params="arm_id
-             robot_ip
-             use_fake_hardware:=^|false
-             fake_sensor_commands:=^|false
-             gazebo:=^|false
-             hand:=^|false
-             gazebo_effort:=^|false
-             arm_prefix:=''
-             multi_arm:=false">
+                 robot_ip
+                 use_fake_hardware:=false
+                 fake_sensor_commands:=false
+                 gazebo:=false
+                 hand:=false
+                 gazebo_effort:=false
+                 arm_prefix:=''">
     <xacro:property name="arm_prefix_modified" value="${'' if arm_prefix == '' else arm_prefix + '_'}" />
     <ros2_control name="${arm_prefix_modified}FrankaHardwareInterface" type="system">
         <hardware>
+          <param name="version">0.1.0</param>
           <param name="arm_id">${arm_id}</param>
           <param name="prefix">${arm_prefix}</param>
@@ -24,15 +24,11 @@
             <plugin>franka_ign_ros2_control/IgnitionSystem</plugin>
           </xacro:if>
-          <xacro:if value="${use_fake_hardware == 0 and gazebo == 0 and multi_arm == 0}">
+          <xacro:if value="${use_fake_hardware == 0 and gazebo == 0}">
             <plugin>franka_hardware/FrankaHardwareInterface</plugin>
             <param name="robot_ip">${robot_ip}</param>
             <param name="arm_prefix">${arm_prefix}</param>
           </xacro:if>
-          <xacro:if value="${use_fake_hardware == 0 and gazebo == 0 and multi_arm == 1}">
-            <plugin>franka_hardware/MultiFrankaHardwareInterface</plugin>
-            <param name="robot_ip">${robot_ip}</param>
-            <param name="arm_prefix">${arm_prefix}</param>
-          </xacro:if>
         </hardware>
+      <!-- Joint position, velocity and effort interfaces -->
       <xacro:macro name="configure_joint" params="joint_name initial_position">
         <joint name="${joint_name}">
@@ -41,8 +37,6 @@
             https://github.com/ros-controls/gz_ros2_control/issues/343
             Command Interfaces -->
-          <xacro:if value="${multi_arm == 0}">
             <command_interface name="position"/>
             <command_interface name="velocity"/>
-          </xacro:if>
           <xacro:if value="${gazebo == 0 or gazebo_effort == 1}">
             <command_interface name="effort"/>
@@ -57,14 +51,38 @@
         </joint>
       </xacro:macro>
-      <xacro:configure_joint joint_name="${arm_prefix_modified}${arm_id}_joint1" initial_position="0.0"/>
-      <xacro:configure_joint joint_name="${arm_prefix_modified}${arm_id}_joint2" initial_position="${-pi/4}"/>
-      <xacro:configure_joint joint_name="${arm_prefix_modified}${arm_id}_joint3" initial_position="0.0"/>
-      <xacro:configure_joint joint_name="${arm_prefix_modified}${arm_id}_joint4" initial_position="${-3*pi/4}"/>
-      <xacro:configure_joint joint_name="${arm_prefix_modified}${arm_id}_joint5" initial_position="0.0"/>
-      <xacro:configure_joint joint_name="${arm_prefix_modified}${arm_id}_joint6" initial_position="${pi/2}"/>
-      <xacro:configure_joint joint_name="${arm_prefix_modified}${arm_id}_joint7" initial_position="${pi/4}"/>
+      <xacro:configure_joint joint_name="${arm_prefix}${arm_id}_joint1" initial_position="0.0"/>
+      <xacro:configure_joint joint_name="${arm_prefix}${arm_id}_joint2" initial_position="${-pi/4}"/>
+      <xacro:configure_joint joint_name="${arm_prefix}${arm_id}_joint3" initial_position="0.0"/>
+      <xacro:configure_joint joint_name="${arm_prefix}${arm_id}_joint4" initial_position="${-3*pi/4}"/>
+      <xacro:configure_joint joint_name="${arm_prefix}${arm_id}_joint5" initial_position="0.0"/>
+      <xacro:configure_joint joint_name="${arm_prefix}${arm_id}_joint6" initial_position="${pi/2}"/>
+      <xacro:configure_joint joint_name="${arm_prefix}${arm_id}_joint7" initial_position="${pi/4}"/>
       <xacro:if value="${gazebo and hand}">
         <xacro:configure_joint joint_name="${arm_id}_finger_joint1" initial_position="0.0" />
       </xacro:if>
+      <xacro:macro name="general_purpose_io" params="prefix command_interface index">
+        <gpio name="${prefix}">
+          <command_interface name="${command_interface}"/>
+          <param name="index">${index}</param>
+        </gpio>
+      </xacro:macro>
+      <!-- Cartesian velocity interfaces -->
+      <xacro:general_purpose_io prefix="vx" command_interface="cartesian_velocity" index="0"/>
+      <xacro:general_purpose_io prefix="vy" command_interface="cartesian_velocity" index="1"/>
+      <xacro:general_purpose_io prefix="vz" command_interface="cartesian_velocity" index="2"/>
+      <xacro:general_purpose_io prefix="wx" command_interface="cartesian_velocity" index="3"/>
+      <xacro:general_purpose_io prefix="wy" command_interface="cartesian_velocity" index="4"/>
+      <xacro:general_purpose_io prefix="wz" command_interface="cartesian_velocity" index="5"/>
+      <!-- Cartesian pose interfaces, in total 16 interfaces -->
+      <xacro:macro name="loop" params="i">
+        <xacro:unless value="${i == 16}">
+          <xacro:general_purpose_io prefix="${i}" command_interface="cartesian_pose_command" index="${i}"/>
+          <xacro:loop i="${i+1}"/>
+        </xacro:unless>
+      </xacro:macro>
+      <xacro:loop i="0"/>
+      <!-- Elbow command interfaces -->
+      <xacro:general_purpose_io prefix="joint_3_position" command_interface="elbow_command" index="0"/>
+      <xacro:general_purpose_io prefix="joint_4_sign" command_interface="elbow_command" index="1"/>
     </ros2_control>
     <xacro:if value="${gazebo}">

File: robots/common/franka_robot.xacro (robot description, xacro)
@@ -10,6 +10,12 @@
                       xyz:='0 0 0'
                       rpy:='0 0 0'
+                      xyz_ee:='0 0 0'
+                      rpy_ee:='0 0 0'
+                      tcp_xyz:='0 0 0'
+                      tcp_rpy:='0 0 0'
+                      safety_distance:='0.03'
                       hand:='true'
                       ee_id:=none
+                      special_connection:=''
                       gazebo:='false'
                       with_sc:='false'
@@ -21,12 +27,11 @@
                       no_prefix:='false'
                       arm_prefix:=''
-                      connected_to:='base'
-                      multi_arm:=false">
+                      description_pkg:='franka_description'
+                      connected_to:='base'">
     <xacro:include filename="$(find franka_description)/robots/common/utils.xacro" />
     <xacro:include filename="$(find franka_description)/robots/common/franka_arm.xacro" />
-    <xacro:property name="arm_prefix_modified" value="${'' if arm_prefix == '' else arm_prefix + '_'}" />
     <xacro:franka_arm
       arm_id="${arm_id}"
-      arm_prefix="${arm_prefix_modified}"
+      arm_prefix="${arm_prefix}"
       no_prefix="${no_prefix}"
       xyz="${xyz}"
@@ -44,9 +49,8 @@
       <xacro:include filename="$(find franka_description)/end_effectors/common/franka_hand.xacro"/>
       <xacro:include filename="$(find franka_description)/end_effectors/common/utils.xacro" />
-      <xacro:include filename="$(find franka_description)/end_effectors/$(arg ee_id)/$(arg ee_id)_arguments.xacro" />
       <xacro:if value="${arm_id == 'fp3'}">
         <xacro:property name="ee_color" value="black" />
       </xacro:if>
-      <xacro:if value="${arm_id == 'fr3' or arm_id == 'fer'}">
+      <xacro:if value="${arm_id == 'fr3' or arm_id == 'fer' or arm_id == 'fr3v2'}">
         <xacro:property name="ee_color" value="white" />
       </xacro:if>
@@ -54,16 +58,16 @@
       <xacro:property name="connection" value="${special_connection if special_connection != '' else arm_id + '_link8'}" />
       <xacro:franka_hand
-        connected_to="${arm_prefix_modified}${connection}"
+        connected_to="${arm_prefix}${connection}"
         arm_id="${arm_id}"
-        arm_prefix="${arm_prefix_modified}"
+        arm_prefix="${arm_prefix}"
         ee_id="${ee_id}_${ee_color}"
-        ee_inertials="${xacro.load_yaml('$(find franka_description)/end_effectors/$(arg ee_id)/inertials.yaml')}"
-        rpy_ee="$(arg rpy_ee)"
-        xyz_ee="$(arg xyz_ee)"
-        tcp_xyz="$(arg tcp_xyz)"
-        tcp_rpy="$(arg tcp_rpy)"
-        safety_distance="$(arg safety_distance)"
+        ee_inertials="${xacro.load_yaml('$(find franka_description)/end_effectors/' + ee_id + '/inertials.yaml')}"
+        rpy_ee="${rpy_ee}"
+        xyz_ee="${xyz_ee}"
+        tcp_xyz="${tcp_xyz}"
+        tcp_rpy="${tcp_rpy}"
+        safety_distance="${safety_distance}"
         gazebo="${gazebo}"
-        description_pkg="$(arg description_pkg)"
+        description_pkg="${description_pkg}"
         with_sc="${with_sc}"
       />
@@ -72,20 +76,19 @@
       <xacro:include filename="$(find franka_description)/end_effectors/common/ee_with_one_link.xacro"/>
       <xacro:include filename="$(find franka_description)/end_effectors/common/utils.xacro" />
-      <xacro:include filename="$(find franka_description)/end_effectors/$(arg ee_id)/$(arg ee_id)_arguments.xacro" />
-      <xacro:property name="special_connection" value="$(arg special_connection)" />
+      <xacro:property name="special_connection" value="${special_connection}" />
       <xacro:property name="connection" value="${special_connection if special_connection == '' else arm_id + '_link8'}" />
       <xacro:ee_with_one_link
-        connected_to="${arm_prefix_modified}${connection}"
+        connected_to="${arm_prefix}${connection}"
         arm_id="${arm_id}"
-        arm_prefix="${arm_prefix_modified}"
+        arm_prefix="${arm_prefix}"
         ee_id="${ee_id}"
-        ee_inertials="${xacro.load_yaml('$(find franka_description)/end_effectors/$(arg ee_id)/inertials.yaml')}"
-        rpy_ee="$(arg rpy_ee)"
-        xyz_ee="$(arg xyz_ee)"
-        tcp_xyz="$(arg tcp_xyz)"
-        tcp_rpy="$(arg tcp_rpy)"
-        safety_distance="$(arg safety_distance)"
+        ee_inertials="${xacro.load_yaml('$(find franka_description)/end_effectors/${ee_id}/inertials.yaml')}"
+        rpy_ee="${rpy_ee}"
+        xyz_ee="${xyz_ee}"
+        tcp_xyz="${tcp_xyz}"
+        tcp_rpy="${tcp_rpy}"
+        safety_distance="${safety_distance}"
         gazebo="${gazebo}"
-        description_pkg="$(arg description_pkg)"
+        description_pkg="${description_pkg}"
         with_sc="${with_sc}"
       />
@@ -143,11 +146,10 @@
           arm_id="${arm_id}"
           robot_ip="${robot_ip}"
-          use_fake_hardware="$(arg use_fake_hardware)"
-          fake_sensor_commands="$(arg fake_sensor_commands)"
-          gazebo="$(arg gazebo)"
-          hand="$(arg hand)"
-          gazebo_effort="$(arg gazebo_effort)"
+          use_fake_hardware="${use_fake_hardware}"
+          fake_sensor_commands="${fake_sensor_commands}"
+          gazebo="${gazebo}"
+          hand="${hand}"
+          gazebo_effort="${gazebo_effort}"
           arm_prefix="${arm_prefix}"
-          multi_arm="$(arg multi_arm)"
       />
     </xacro:if>

File: robots/fer/fer.urdf.xacro (robot description, xacro)
@@ -8,4 +8,6 @@
   -->
   <xacro:arg name="arm_id" default="fer" />
+  <!-- The prefix of the robot -->
+  <xacro:arg name="arm_prefix" default="" />
   <!-- Don't print a prefix for joints, visuals, and links? -->
   <xacro:arg name="no_prefix" default="false"/>
@@ -14,12 +16,16 @@
   <!-- Which end-effector would be mounted at the flange?" -->
   <xacro:arg name="ee_id" default="franka_hand" />
-  <!-- Is the robot being simulated in gazebo?" -->
-  <xacro:arg name="gazebo" default="false" />
-  <!-- If `gazebo` arg is set, to which frame shall $(arm_id)_link0 be parented. Empty string for not fixing at all -->
-  <xacro:arg name="parent" default="world" />
-  <!-- If `gazebo` arg is set and `parent` not empty, what position offset between `parent` & $(arm_id)_link0 -->
-  <xacro:arg name="xyz" default="0 0 0" />
-  <!-- If `gazebo` arg is set and `parent` not empty, what rotation offset between `parent` & $(arm_id)_link0 -->
-  <xacro:arg name="rpy" default="0 0 0" />
+  <!-- Where is the end-effector connected to, if different from the robot flange?  -->
+  <xacro:arg name="special_connection" default="" />
+  <!-- Position offset between ee and parent frame -->
+  <xacro:arg name="xyz_ee" default="0 0 0" />
+  <!-- Rotation offset between ee and parent frame -->
+  <xacro:arg name="rpy_ee" default= "0 0 ${-pi/4}" />
+  <!-- Position offset between ee frame and tcp frame -->
+  <xacro:arg name="tcp_xyz" default="0 0 0.1034" />
+  <!-- Rotation offset between ee frame and tcp frame -->
+  <xacro:arg name="tcp_rpy" default="0 0 0" />
+  <!-- Safety distance for the collision capsules -->
+  <xacro:arg name="safety_distance" default="0.03" />
   <!-- Should self-collision be enabled? -->
   <xacro:arg name="with_sc" default="false" />
@@ -32,8 +38,13 @@
   <!-- Should fake sensors be used? -->
   <xacro:arg name="fake_sensor_commands" default="false" />
+  <!-- Should the robot be spawned in Gazebo?" -->
+  <xacro:arg name="gazebo" default="false" />
   <!-- Should the robot be spawned in Gazebo with effort interfaces?" -->
   <xacro:arg name="gazebo_effort" default="false" />
-  <!-- For a multi arm setup, we need a threaded robot running async-->
-  <xacro:arg name="multi_arm" default="false" />
+  <!-- Name of the description package -->
+  <xacro:arg name="description_pkg" default="franka_description" />
+  <!-- Append an underscore to the user-provided prefix, if non-empty. -->
+  <xacro:property name="prefix" value="$(arg arm_prefix)"/>
+  <xacro:property name="modified_prefix" value="${prefix + '_' if prefix else ''}"/>
   <xacro:franka_robot arm_id="fer"
                       joint_limits="${xacro.load_yaml('$(find franka_description)/robots/fer/joint_limits.yaml')}"
@@ -44,4 +55,10 @@
                       hand="$(arg hand)"
                       ee_id="$(arg ee_id)"
+                      special_connection="$(arg special_connection)"
+                      xyz_ee="$(arg xyz_ee)"
+                      rpy_ee="$(arg rpy_ee)"
+                      tcp_xyz="$(arg tcp_xyz)"
+                      tcp_rpy="$(arg tcp_rpy)"
+                      safety_distance="$(arg safety_distance)"
                       with_sc="$(arg with_sc)"
                       ros2_control="$(arg ros2_control)"
@@ -51,5 +68,6 @@
                       gazebo_effort="$(arg gazebo_effort)"
                       no_prefix="$(arg no_prefix)"
-                      arm_prefix= ""
+                      arm_prefix="${modified_prefix}"
+                      description_pkg="$(arg description_pkg)"
                       connected_to= "base">
   </xacro:franka_robot>

File: robots/fp3/fp3.urdf.xacro (robot description, xacro)
@@ -8,4 +8,6 @@
   -->
   <xacro:arg name="arm_id" default="fp3" />
+  <!-- The prefix of the robot -->
+  <xacro:arg name="arm_prefix" default="" />
   <!-- Don't print a prefix for joints, visuals, and links? -->
   <xacro:arg name="no_prefix" default="false"/>
@@ -14,4 +16,16 @@
   <!-- Which end-effector would be mounted at the flange?" -->
   <xacro:arg name="ee_id" default="franka_hand" />
+  <!-- Where is the end-effector connected to, if different from the robot flange?  -->
+  <xacro:arg name="special_connection" default="" />
+  <!-- Position offset between ee and parent frame -->
+  <xacro:arg name="xyz_ee" default="0 0 0" />
+  <!-- Rotation offset between ee and parent frame -->
+  <xacro:arg name="rpy_ee" default= "0 0 ${-pi/4}" />
+  <!-- Position offset between ee frame and tcp frame -->
+  <xacro:arg name="tcp_xyz" default="0 0 0.1034" />
+  <!-- Rotation offset between ee frame and tcp frame -->
+  <xacro:arg name="tcp_rpy" default="0 0 0" />
+  <!-- Safety distance for the collision capsules -->
+  <xacro:arg name="safety_distance" default="0.03" />
   <!-- Should self-collision be enabled? -->
   <xacro:arg name="with_sc" default="false" />
@@ -28,6 +42,9 @@
   <!-- Should the robot be spawned in Gazebo with effort interfaces?" -->
   <xacro:arg name="gazebo_effort" default="false" />
-  <!-- For a multi arm setup, we need a threaded robot running async-->
-  <xacro:arg name="multi_arm" default="false" />
+  <!-- Name of the description package -->
+  <xacro:arg name="description_pkg" default="franka_description" />
+  <!-- Append an underscore to the user-provided prefix, if non-empty. -->
+  <xacro:property name="prefix" value="$(arg arm_prefix)"/>
+  <xacro:property name="modified_prefix" value="${prefix + '_' if prefix else ''}"/>
   <xacro:franka_robot arm_id="fp3"
                       joint_limits="${xacro.load_yaml('$(find franka_description)/robots/fp3/joint_limits.yaml')}"
@@ -38,4 +55,10 @@
                       hand="$(arg hand)"
                       ee_id="$(arg ee_id)"
+                      special_connection="$(arg special_connection)"
+                      xyz_ee="$(arg xyz_ee)"
+                      rpy_ee="$(arg rpy_ee)"
+                      tcp_xyz="$(arg tcp_xyz)"
+                      tcp_rpy="$(arg tcp_rpy)"
+                      safety_distance="$(arg safety_distance)"
                       with_sc="$(arg with_sc)"
                       ros2_control="$(arg ros2_control)"
@@ -45,5 +68,6 @@
                       gazebo_effort="$(arg gazebo_effort)"
                       no_prefix="$(arg no_prefix)"
-                      arm_prefix= ""
+                      arm_prefix="${modified_prefix}"
+                      description_pkg="$(arg description_pkg)"
                       connected_to= "base">
   </xacro:franka_robot>
