Commit message: Imported upstream version '1.0.1' of 'upstream'

File: robots/fr3/fr3.urdf.xacro (robot description, xacro)
@@ -8,4 +8,6 @@
   -->
   <xacro:arg name="arm_id" default="fr3" />
+  <!-- The prefix of the robot -->
+  <xacro:arg name="arm_prefix" default="" />
   <!-- Don't print a prefix for joints, visuals, and links? -->
   <xacro:arg name="no_prefix" default="false"/>
@@ -14,4 +16,16 @@
   <!-- Which end-effector would be mounted at the flange?" -->
   <xacro:arg name="ee_id" default="franka_hand" />
+  <!-- Where is the end-effector connected to, if different from the robot flange?  -->
+  <xacro:arg name="special_connection" default="" />
+  <!-- Position offset between ee and parent frame -->
+  <xacro:arg name="xyz_ee" default="0 0 0" />
+  <!-- Rotation offset between ee and parent frame -->
+  <xacro:arg name="rpy_ee" default= "0 0 ${-pi/4}" />
+  <!-- Position offset between ee frame and tcp frame -->
+  <xacro:arg name="tcp_xyz" default="0 0 0.1034" />
+  <!-- Rotation offset between ee frame and tcp frame -->
+  <xacro:arg name="tcp_rpy" default="0 0 0" />
+  <!-- Safety distance for the collision capsules -->
+  <xacro:arg name="safety_distance" default="0.03" />
   <!-- Should self-collision be enabled? -->
   <xacro:arg name="with_sc" default="false" />
@@ -28,6 +42,9 @@
   <!-- Should the robot be spawned in Gazebo with effort interfaces?" -->
   <xacro:arg name="gazebo_effort" default="false" />
-  <!-- For a multi arm setup, we need a threaded robot running async-->
-  <xacro:arg name="multi_arm" default="false" />
+  <!-- Name of the description package -->
+  <xacro:arg name="description_pkg" default="franka_description" />
+  <!-- Append an underscore to the user-provided prefix, if non-empty. -->
+  <xacro:property name="prefix" value="$(arg arm_prefix)"/>
+  <xacro:property name="modified_prefix" value="${prefix + '_' if prefix else ''}"/>
   <xacro:franka_robot arm_id="fr3"
                       joint_limits="${xacro.load_yaml('$(find franka_description)/robots/fr3/joint_limits.yaml')}"
@@ -38,4 +55,10 @@
                       hand="$(arg hand)"
                       ee_id="$(arg ee_id)"
+                      special_connection="$(arg special_connection)"
+                      xyz_ee="$(arg xyz_ee)"
+                      rpy_ee="$(arg rpy_ee)"
+                      tcp_xyz="$(arg tcp_xyz)"
+                      tcp_rpy="$(arg tcp_rpy)"
+                      safety_distance="$(arg safety_distance)"
                       with_sc="$(arg with_sc)"
                       ros2_control="$(arg ros2_control)"
@@ -45,5 +68,6 @@
                       gazebo_effort="$(arg gazebo_effort)"
                       no_prefix="$(arg no_prefix)"
-                      arm_prefix= ""
+                      arm_prefix="${modified_prefix}"
+                      description_pkg="$(arg description_pkg)"
                       connected_to= "base">
   </xacro:franka_robot>
